File: PDB_ESC_BEC.sch (EAGLE design)
At the start: 50 parts, among them IC1 STM32F10XCXT6, Q1 N-HEXFET-2D_SOT232-, Q2 N-HEXFET-2D_SOT232-, Q3 N-HEXFET-2D_SOT232-, Q6 N-HEXFET-2D_SOT232-, U1 TPS61200, X1 87438-02, X2 87438-02, X3 87438-02, X4 87438-02

Commit message: Added files via upload
Connections:
- removed net JDTI: TP2.P$1
- net JTDI: now also TP2.P$1
Changed lines of the file:
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@@
 <pinref part="U$2" gate="-CAN_GND" pin="S"/>
 <wire x1="-147.32" y1="10.16" x2="-147.32" y2="17.78" width="0.1524" layer="91"/>
+<junction x="-170.18" y="15.24"/>
 </segment>
 <segment>
@@
 <pinref part="TP3" gate="G$1" pin="P$1"/>
 <wire x1="-27.94" y1="15.24" x2="-30.48" y2="15.24" width="0.1524" layer="91"/>
-<label x="-40.64" y="15.24" size="1.778" layer="95"/>
+<label x="-38.1" y="15.24" size="1.778" layer="95"/>
 </segment>
 <segment>
@@
 </segment>
 </net>
-<net name="JDTI" class="0">
-<segment>
-<pinref part="TP2" gate="G$1" pin="P$1"/>
-<wire x1="-27.94" y1="7.62" x2="-30.48" y2="7.62" width="0.1524" layer="91"/>
-<label x="-38.1" y="7.62" size="1.778" layer="95"/>
-</segment>
-</net>
 <net name="JTDO" class="0">
 <segment>
 <pinref part="TP1" gate="G$1" pin="P$1"/>
 <wire x1="-27.94" y1="0" x2="-30.48" y2="0" width="0.1524" layer="91"/>
-<label x="-40.64" y="0" size="1.778" layer="95"/>
+<label x="-38.1" y="0" size="1.778" layer="95"/>
 </segment>
 <segment>
@@
 <label x="-345.44" y="-71.12" size="1.778" layer="95"/>
 </segment>
-</net>
+<segment>
+<pinref part="TP2" gate="G$1" pin="P$1"/>
+<wire x1="-27.94" y1="7.62" x2="-30.48" y2="7.62" width="0.1524" layer="91"/>
+<label x="-38.1" y="7.62" size="1.778" layer="95"/>
+</segment>
+</net>

Commit message: Added files via upload
Parts:
- removed R11, R5, R7: 10k, eagle-ltspice:R0204/7
- removed R12, R4, R6, R8: 1M, eagle-ltspice:R0204/7
- removed TP1, TP2, TP3, TP4, TP5, TP6, TP7: PAD-POGO, pixhawk2:PAD-POGO
- added C11: 10n, pixhawk2:CAP1206
- added C12: 1u, pixhawk2:CAP1206
- added C13: 4.7u, pixhawk2:CAP1206
- added R15, R18, R20, R22: 10K, pixhawk2:RESISTOR1206
- added R16, R17, R19, R21: 100K, pixhawk2:RESISTOR1206
- added U$3, U$4, U$5, U$6: MOUNT-HOLE3.1MM, pixhawk2:MOUNT-HOLE3.1MM
- added X5: SM06B-SRSS-TB, con-jst2:SM06B-SRSS-TB
- C10, C8, C9: value 100p -> 100n
- D1: value (none) -> 5V
- R3: value 10k -> 120; device eagle-ltspice:R0204/7 -> pixhawk2:RESISTOR1206; PROD_ID RES-00824 -> (none)
- R9: value (none) -> 10K
Connections:
- net IO_BOOT0 renamed BOOT0
- net N$15 renamed BOOT1
- removed net NJTRST: IC1PORTB_L.PB4, TP4.P$1
- net GND: now also C11.2, C12.2, C13.1, R16.2, R17.1, R19.1, R21.2, X5-6.S; no longer R12.2, R4.2, R6.2, R8.2, TP6.P$1
- net JTCLK: now also X5-5.S; no longer TP3.P$1
- net JTDI: now also X5-3.S; no longer TP2.P$1
- net JTDO: now also X5-2.S; no longer TP1.P$1
- net JTMS: now also X5-4.S; no longer TP5.P$1
- net N$10: now also R3.2
- net N$13: now also R3.1
- net N$3: now also R21.1, R22.2; no longer R3.2, R4.1
- net N$5: now also R17.2, R18.1; no longer R5.2, R6.1
- net N$6: now also R15.2, R16.1; no longer R11.2, R12.1
- net N$8: now also R19.2, R20.1; no longer R7.2, R8.1
- net TIM1_CH1N: now also R15.1; no longer R11.1
- net TIM1_CH2N: now also R22.1; no longer R3.1
- net TIM1_CH3N: now also R20.2; no longer R7.1
- net TIM1_CH4N: now also R18.2; no longer R5.1
- net VBAT: no longer IC1AN_POWER.VBAT
- net VCC_3.3V_1: now also C11.1, C12.1, C13.2, IC1AN_POWER.VBAT, X5-1.S; no longer TP7.P$1
Other:
- moved on the sheet: C10, C9, IC1AN_POWER, IC1PORTA_H, IC1PORTA_L, IC1PORTB_H, IC1PORTD/OSC
